Commit message: testing autonomy

File: stinger_description/urdf/stinger_tug.urdf (robot description, URDF)
Before this commit: robot stinger_tug, 6 links, 5 joints
Joints:
- joint imu_joint: origin xyz=0 0 0 rpy=0 0 0 -> xyz=0 0 0 rpy=0 3.141 0

Commit message: launch & urdf & filter  changes

File: stinger_description/urdf/stinger_tug.urdf (robot description, URDF)
Before this commit: robot stinger_tug, 6 links, 5 joints
Links:
- removed link laser_frame
- added link laser, mass 0.1; collision cylinder length=0.04 radius=0.05; visual cylinder length=0.04 radius=0.05
Joints:
- joint lidar_joint: child laser_frame -> laser
