Commit message: Add IMU and GPS to sim

File: stinger_description/models/stinger_base/components/sensors.xacro (robot description, xacro)
@@ -5,5 +5,5 @@
     <joint name="camera_joint_${camera_id}" type="fixed">
       <xacro:insert_block name="origin"/>
-      <parent link="base_link"/>
+      <parent link="hull_link"/>
       <child link="camera_${camera_id}"/>
       <axis xyz="1 0 0"/>
@@ -33,5 +33,5 @@
     <joint name="lidar_joint" type="fixed">
       <xacro:insert_block name="origin"/>
-      <parent link="base_link"/>
+      <parent link="hull_link"/>
       <child link="lidar"/>
       <axis xyz="1 0 0"/>
@@ -62,5 +62,5 @@
         <update_rate>10</update_rate>
         <visualize>true</visualize>
-        <topic>stinger/scan</topic>
+        <topic>stinger/laser/scan</topic>
         <!-- This tag isn't recognized by SDF but is extremely important for getting the correct TF data for the sonar frame-->
         <gz_frame_id>lidar</gz_frame_id>
@@ -68,3 +68,39 @@
     </gazebo>
   </xacro:macro>
+  <xacro:macro name="imu_macro" params="*origin">
+    <link name="imu"/>
+    <joint name="imu_joint" type="fixed">
+      <xacro:insert_block name="origin"/>
+      <parent link="hull_link"/>
+      <child link="imu"/>
+      <axis xyz="1 0 0"/>
+    </joint>
+    <gazebo reference="imu">
+      <sensor name="imu_sensor" type="imu">
+        <pose>0 0 0 0 0 0</pose>
+        <always_on>1</always_on>
+        <topic>stinger/imu/data</topic>
+        <enable_metrics>true</enable_metrics>
+        <update_rate>1000</update_rate>
+        <!-- This tag isn't recognized by SDF but is extremely important for getting the correct TF data for the IMU frame-->
+        <gz_frame_id>imu</gz_frame_id>
+      </sensor>
+    </gazebo>
+  </xacro:macro>
+  <xacro:macro name="gps_macro" params="*origin">
+    <link name="gps_link"/>
+    <joint name="gps_joint" type="fixed">
+      <xacro:insert_block name="origin"/>
+      <parent link="hull_link"/>
+      <child link="gps_link"/>
+    </joint>
+    <gazebo reference="gps_link">
+      <sensor name="gps_sensor" type="navsat">
+        <always_on>1</always_on>
+        <update_rate>10</update_rate>
+        <topic>stinger/gps/fix</topic>
+        <gz_frame_id>gps</gz_frame_id>
+      </sensor>
+    </gazebo>
+  </xacro:macro>
 </robot>

File: stinger_description/models/stinger_base/stinger_base.xacro (robot description, xacro)
@@ -6,5 +6,5 @@
     <link name="hull_link">
       <inertial>
-        <pose>0.0 0.0 -0.2 0 0 0</pose>
+        <pose>0.0 0.0 -0.13 0 0 0</pose>
         <mass value="5"/>
         <inertia ixx="2.42369" ixy="0" ixz="0" iyy="3.9235025" iyz="0" izz="5.6403125"/>
@@ -89,33 +89,10 @@
       <origin xyz="0.1 0 0.025" rpy="0 0 0" />
     </xacro:lidar_macro>
-    <link name="imu_link">
-      <inertial>
-        <pose>0.1 0 0 0 0 0</pose>
-        <mass value="0.1"/>
-        <inertia ixx="0.0001" ixy="0" ixz="0" iyy="0.0001" iyz="0" izz="0.0001" />
-      </inertial>
-      <sensor name="imu_sensor" type="imu">
-        <pose degrees="true">0 0 0 180 0 0</pose>
-        <always_on>1</always_on>
-        <update_rate>1000.0</update_rate>
-      </sensor>
-    </link>
-    <joint name="imu_joint" type="fixed">
-      <origin xyz="0 0 0"/>
-      <parent link="hull_link"/>
-      <child link="imu_link"/>
-    </joint>
-    <link name="gps_link">
-      <sensor name="gps_sensor" type="gps">
-        <pose degrees="true">0 0 0 180 0 0</pose>
-        <always_on>1</always_on>
-        <update_rate>1000.0</update_rate>
-      </sensor>
-    </link>
-    <joint name="gps_joint" type="fixed">
-      <origin xyz="0 0 0"/>
-      <parent link="hull_link"/>
-      <child link="gps_link"/>
-    </joint>
+    <xacro:imu_macro>
+      <origin xyz="-0.05 0 0.025" rpy="0 0 0" />
+    </xacro:imu_macro>
+    <xacro:gps_macro>
+      <origin xyz="-0.05 0 0.025" rpy="0 0 0" />
+    </xacro:gps_macro>
     <!-- hydrodynamics and control plugins -->
     <gazebo>
@@ -141,5 +118,4 @@
         <mQabsQ>-60</mQabsQ>
         <nRabsR>-50</nRabsR>
-        <default_current> 0.025 -0.025 0.5</default_current>
       </plugin>
     </gazebo>
