Commit message: Prefix stinger frames
Fixed issue with type for use_sim_time

Made changes to topic prefix conventions

File: stinger_description/models/stinger_base/components/sensors.xacro (robot description, xacro)
@@ -1,13 +1,13 @@
 <?xml version="1.0"?>
 <robot xmlns:xacro="http://www.ros.org/wiki/xacro">
- <xacro:macro name="camera_macro" params="camera_id *origin">
-    <link name="camera_${camera_id}"/>
-    <joint name="camera_joint_${camera_id}" type="fixed">
+ <xacro:macro name="camera_macro" params="prefix topic_prefix camera_id *origin">
+   <link name="${prefix}camera_${camera_id}"/>
+   <joint name="${prefix}camera_joint_${camera_id}" type="fixed">
       <xacro:insert_block name="origin"/>
-      <parent link="hull_link"/>
-      <child link="camera_${camera_id}"/>
+      <parent link="${prefix}hull_link"/>
+      <child link="${prefix}camera_${camera_id}"/>
       <axis xyz="1 0 0"/>
     </joint>
-    <gazebo reference="camera_${camera_id}">
+    <gazebo reference="${prefix}camera_${camera_id}">
       <sensor name="camera_${camera_id}" type="camera">
         <camera>
@@ -25,17 +25,17 @@
         <update_rate>10</update_rate>
         <visualize>true</visualize>
-        <topic>stinger/camera_${camera_id}/image_raw</topic>
+        <topic>/${topic_prefix}/camera_${camera_id}/image_raw</topic>
       </sensor>
     </gazebo>
   </xacro:macro>
-  <xacro:macro name="lidar_macro" params="*origin">
-    <link name="lidar"/>
-    <joint name="lidar_joint" type="fixed">
+  <xacro:macro name="lidar_macro" params="prefix topic_prefix *origin">
+    <link name="${prefix}lidar"/>
+    <joint name="${prefix}lidar_joint" type="fixed">
       <xacro:insert_block name="origin"/>
-      <parent link="hull_link"/>
-      <child link="lidar"/>
+      <parent link="${prefix}hull_link"/>
+      <child link="${prefix}lidar"/>
       <axis xyz="1 0 0"/>
     </joint>
-    <gazebo reference="lidar">
+    <gazebo reference="${prefix}lidar">
       <sensor name="lidar" type="gpu_lidar">
         <lidar>
@@ -62,42 +62,42 @@
         <update_rate>10</update_rate>
         <visualize>true</visualize>
-        <topic>stinger/laser/scan</topic>
-        <gz_frame_id>lidar</gz_frame_id>
+        <topic>/${topic_prefix}/laser/scan</topic>
+        <gz_frame_id>${prefix}lidar</gz_frame_id>
       </sensor>
     </gazebo>
   </xacro:macro>
-  <xacro:macro name="imu_macro" params="*origin">
-    <link name="imu_link"/>
-    <joint name="imu_joint" type="fixed">
+  <xacro:macro name="imu_macro" params="prefix topic_prefix *origin">
+    <link name="${prefix}imu_link"/>
+    <joint name="${prefix}imu_joint" type="fixed">
       <xacro:insert_block name="origin"/>
-      <parent link="base_link"/>
-      <child link="imu_link"/>
+      <parent link="${prefix}base_link"/>
+      <child link="${prefix}imu_link"/>
       <axis xyz="1 0 0"/>
     </joint>
-    <gazebo reference="imu_link">
+    <gazebo reference="${prefix}imu_link">
       <sensor name="imu_sensor" type="imu">
         <pose>0 0 0 0 0 0</pose>
         <always_on>1</always_on>
-        <topic>stinger/imu/data</topic>
+        <topic>/${topic_prefix}/imu/data</topic>
         <enable_metrics>true</enable_metrics>
         <update_rate>100</update_rate>
         <!-- This tag isn't recognized by SDF but is extremely important for getting the correct TF data for the IMU frame-->
-        <gz_frame_id>imu_link</gz_frame_id>
+        <gz_frame_id>${prefix}imu_link</gz_frame_id>
       </sensor>
     </gazebo>
   </xacro:macro>
-  <xacro:macro name="gps_macro" params="*origin">
-    <link name="gps_link"/>
-    <joint name="gps_joint" type="fixed">
+  <xacro:macro name="gps_macro" params="prefix topic_prefix *origin">
+    <link name="${prefix}gps_link"/>
+    <joint name="${prefix}gps_joint" type="fixed">
       <xacro:insert_block name="origin"/>
-      <parent link="hull_link"/>
-      <child link="gps_link"/>
+      <parent link="${prefix}hull_link"/>
+      <child link="${prefix}gps_link"/>
     </joint>
-    <gazebo reference="gps_link">
+    <gazebo reference="${prefix}gps_link">
       <sensor name="gps_sensor" type="navsat">
         <always_on>1</always_on>
         <update_rate>10</update_rate>
-        <topic>stinger/gps/fix</topic>
-        <gz_frame_id>gps_link</gz_frame_id>
+        <topic>/${topic_prefix}/gps/fix</topic>
+        <gz_frame_id>${prefix}gps_link</gz_frame_id>
       </sensor>
     </gazebo>

File: stinger_description/models/stinger_base/components/thrusters.xacro (robot description, xacro)
@@ -2,13 +2,13 @@
 <robot xmlns:xacro="http://www.ros.org/wiki/xacro">
   <xacro:property name="prop_mesh" value="file://$(find stinger_description)/models/stinger_base/meshes/stinger_prop.dae"/>
-  <xacro:macro name="prop_macro" params="thruster_id *origin">
-    <link name="thruster_${thruster_id}"/>
-    <joint name="thruster_joint_${thruster_id}" type="fixed">
+  <xacro:macro name="prop_macro" params="prefix thruster_id *origin">
+    <link name="${prefix}thruster_${thruster_id}"/>
+    <joint name="${prefix}thruster_joint_${thruster_id}" type="fixed">
       <xacro:insert_block name="origin"/>
-      <parent link="base_link"/>
-      <child link="thruster_${thruster_id}"/>
+      <parent link="${prefix}base_link"/>
+      <child link="${prefix}thruster_${thruster_id}"/>
       <axis xyz="1 0 0"/>
     </joint>
-    <link name="propeller_${thruster_id}">
+    <link name="${prefix}propeller_${thruster_id}">
       <!-- The inertial values need to be reasonable or gazebo will crash -->
       <inertial>
@@ -24,7 +24,7 @@
       </visual>
     </link>
-    <joint name="prop_joint_${thruster_id}" type="continuous">
-      <parent link="thruster_${thruster_id}"/>
-      <child link="propeller_${thruster_id}"/>
+    <joint name="${prefix}prop_joint_${thruster_id}" type="continuous">
+      <parent link="${prefix}thruster_${thruster_id}"/>
+      <child link="${prefix}propeller_${thruster_id}"/>
       <axis xyz="1 0 0"/>
     </joint>
@@ -34,5 +34,5 @@
         filename="gz-sim-thruster-system"
         name="gz::sim::systems::Thruster">
-        <joint_name>prop_joint_${thruster_id}</joint_name>
+        <joint_name>${prefix}prop_joint_${thruster_id}</joint_name>
         <thrust_coefficient>0.005</thrust_coefficient>
         <fluid_density>1000</fluid_density>

File: stinger_description/models/stinger_base/stinger_base.xacro (robot description, xacro)
@@ -3,6 +3,6 @@
     <xacro:include filename="$(find stinger_description)/models/stinger_base/components/sensors.xacro"/>
     <xacro:include filename="$(find stinger_description)/models/stinger_base/components/thrusters.xacro"/>
-    <xacro:macro name="stinger_base">
-    <link name="hull_link">
+    <xacro:macro name="stinger_base" params="prefix topic_prefix">
+    <link name="${prefix}hull_link">
       <inertial>
         <pose>0.0 0.0 -0.13 0 0 0</pose>
@@ -18,5 +18,5 @@
     </link>
     <!-- port hull -->
-    <link name="hull_port_link">
+    <link name="${prefix}hull_port_link">
       <inertial>
         <mass value="1.0"/>
@@ -37,11 +37,11 @@
       </collision>
     </link>
-    <joint name="hull_port_joint" type="fixed">
+    <joint name="${prefix}hull_port_joint" type="fixed">
       <origin xyz="0.0 0.0765 -0.035"/>
-      <parent link="hull_link"/>
-      <child link="hull_port_link"/>
+      <parent link="${prefix}hull_link"/>
+      <child link="${prefix}hull_port_link"/>
     </joint>
     <!-- starboard hull -->
-    <link name="hull_stbd_link">
+    <link name="${prefix}hull_stbd_link">
       <inertial>
         <mass value="1.0"/>
@@ -62,27 +62,27 @@
       </collision>
     </link>
-    <joint name="hull_stbd_joint" type="fixed">
+    <joint name="${prefix}hull_stbd_joint" type="fixed">
       <origin xyz="0.0 -0.0765 -0.035"/>
-      <parent link="hull_link"/>
-      <child link="hull_stbd_link"/>
+      <parent link="${prefix}hull_link"/>
+      <child link="${prefix}hull_stbd_link"/>
     </joint>
     <!-- Thrusters -->
-    <xacro:prop_macro thruster_id="port">
+    <xacro:prop_macro prefix="${prefix}" thruster_id="port">
       <origin xyz="-0.19 0.073 -0.041" rpy="0 0 0" />
     </xacro:prop_macro>
-    <xacro:prop_macro thruster_id="stbd">
+    <xacro:prop_macro prefix="${prefix}" thruster_id="stbd">
       <origin xyz="-0.19 -0.073 -0.041" rpy="0 0 0" />
     </xacro:prop_macro>
     <!-- Sensors -->
-    <xacro:camera_macro camera_id="0">
+    <xacro:camera_macro prefix="${prefix}" topic_prefix="${topic_prefix}" camera_id="0">
       <origin xyz="0.16 0 0.012" rpy="0 0 0" />
     </xacro:camera_macro>
-    <xacro:lidar_macro>
+    <xacro:lidar_macro prefix="${prefix}" topic_prefix="${topic_prefix}">
       <origin xyz="0.1 0 0.1" rpy="0 0 0" />
     </xacro:lidar_macro>
-    <xacro:imu_macro>
+    <xacro:imu_macro prefix="${prefix}" topic_prefix="${topic_prefix}">
       <origin xyz="-0.05 0 0.025" rpy="3.14 0 0" />
     </xacro:imu_macro>
-    <xacro:gps_macro>
+    <xacro:gps_macro prefix="${prefix}" topic_prefix="${topic_prefix}">
       <origin xyz="-0.05 0 0.025" rpy="0 0 0" />
     </xacro:gps_macro>
@@ -92,5 +92,5 @@
         filename="gz-sim-hydrodynamics-system"
         name="gz::sim::systems::Hydrodynamics">
-        <link_name> base_link </link_name>
+        <link_name>${prefix}base_link</link_name>
         <!-- Linear Drag -->
         <xU>-5</xU> <!-- Surge -->

File: stinger_description/urdf/stinger_tug.urdf.xacro (robot description, xacro)
@@ -1,12 +1,17 @@
 <?xml version="1.0" ?>
 <robot xmlns:xacro="http://www.ros.org/wiki/xacro" name="stinger_tug">
+  <xacro:arg name="prefix" default=""/>
+  <xacro:arg name="namespace" default="$(arg prefix)"/>
+  <xacro:arg name="topic_prefix" default="stinger"/>
   <xacro:include filename="$(find stinger_description)/models/stinger_base/stinger_base.xacro"/>
-  <link name="base_link">
+  <link name="$(arg namespace)base_link">
   </link>
-  <xacro:stinger_base />
-  <joint name="hull_joint" type="fixed">
+  <xacro:stinger_base
+    prefix="$(arg namespace)"
+    topic_prefix="$(arg topic_prefix)"/>
+  <joint name="$(arg namespace)hull_joint" type="fixed">
     <origin xyz="0 0 0"/>
-    <parent link="base_link"/>
-    <child link="hull_link"/>
+    <parent link="$(arg namespace)base_link"/>
+    <child link="$(arg namespace)hull_link"/>
   </joint>
 </robot>
