Commit message: Add working robot description node, spawning robot still broken

File: stinger_description/models/stinger_base/stinger_base.xacro (robot description, xacro)
@@ -1,4 +1,13 @@
 <?xml version="1.0"?>
 <robot xmlns:xacro="http://www.ros.org/wiki/xacro" name="stinger_base">
+    <material name="white">
+      <color rgba="1 1 1 1"/>
+    </material>
+    <material name="blue">
+      <color rgba="0 0 1 1"/>
+    </material>
+    <material name="red">
+      <color rgba="1 0 0 1"/>
+    </material>
     <xacro:macro name="stinger_base">
     <link name="hull_link">
@@ -14,17 +23,17 @@
           </geometry>
       </collision>
-      <visual name="hull_visual">
+      <!-- <visual name="hull_visual">
         <geometry>
-          <mesh filename="package://stinger_description/models/stinger_base/meshes/stinger_hull.dae"/>
+          <mesh filename="file://$(find stinger_description)/models/stinger_base/meshes/stinger_hull.dae"/>
         </geometry>
-      </visual>
+      </visual> -->
       <visual name="motor_stbd_visual">
         <geometry>
-          <mesh filename="package://stinger_description/models/stinger_base/meshes/stinger_prop.dae"/>
+          <mesh filename="file://$(find stinger_description)/models/stinger_base/meshes/stinger_prop.dae"/>
         </geometry>
       </visual>
       <visual name="motor_port_visual">
         <geometry>
-          <mesh filename="package://stinger_description/models/stinger_base/meshes/stinger_prop.dae"/>
+          <mesh filename="file://$(find stinger_description)/models/stinger_base/meshes/stinger_prop.dae"/>
         </geometry>
       </visual>
@@ -51,7 +60,7 @@
             </geometry>
         </collision>
-        <xacro:inertial_box mass="0.1" x="0.12" y="0.15" z="0.15">
+        <!-- <xacro:inertial_box mass="0.1" x="0.12" y="0.15" z="0.15">
             <origin xyz="0.0 0 0" rpy="0 0 0"/>
-        </xacro:inertial_box>
+        </xacro:inertial_box> -->
     </link>
     <joint name="camera_joint" type="fixed">
@@ -60,5 +69,5 @@
         <child link="camera_link"/>
     </joint>
-    <link name="laser_frame">
+    <link name="lidar_link">
         <visual>
             <geometry>
@@ -72,7 +81,7 @@
             </geometry>
         </collision>
-        <xacro:inertial_cylinder mass="0.1" length="0.04" radius="0.05">
+        <!-- <xacro:inertial_cylinder mass="0.1" length="0.04" radius="0.05">
             <origin xyz="0 0 0" rpy="0 0 0"/>
-        </xacro:inertial_cylinder>
+        </xacro:inertial_cylinder> -->
     </link>
     <joint name="lidar_joint" type="fixed">

Commit message: Add graded buoyancy and hydrodynamic forces

File: stinger_description/models/stinger_base/stinger_base.xacro (robot description, xacro)
@@ -14,19 +14,19 @@
       <inertial>
         <pose>-0.05 0 -0.15 0 0 0</pose>
-        <mass value="30"/>
+        <mass value="7"/>
         <inertia ixx="2.42369" ixy="0" ixz="0" iyy="3.9235025" iyz="0" izz="5.6403125"/>
       </inertial>
       <collision>
-          <origin xyz="0 0 0.05" rpy="0 0 0"/>
+          <origin xyz="0 0 -0.1" rpy="0 0 0"/>
           <geometry>
                 <box size="0.381 0.204 0.135" />
           </geometry>
       </collision>
-      <!-- <visual name="hull_visual">
+      <visual name="hull_visual">
         <geometry>
           <mesh filename="file://$(find stinger_description)/models/stinger_base/meshes/stinger_hull.dae"/>
         </geometry>
-      </visual> -->
-      <visual name="motor_stbd_visual">
+      </visual>
+      <!-- <visual name="motor_stbd_visual">
         <geometry>
           <mesh filename="file://$(find stinger_description)/models/stinger_base/meshes/stinger_prop.dae"/>
@@ -37,27 +37,7 @@
           <mesh filename="file://$(find stinger_description)/models/stinger_base/meshes/stinger_prop.dae"/>
         </geometry>
-      </visual>
+      </visual> -->
     </link>
     <link name="camera_link">
-        <visual>
-            <origin xyz="-0.03 0 0" rpy="0 0 0"/>
-            <geometry>
-                <box size="0.06 0.15 0.15" />
-            </geometry>
-            <material name="white" />
-        </visual>
-        <visual>
-            <origin xyz="0.03 0 0" rpy="0 ${pi/2} 0"/>
-            <geometry>
-                <cylinder length="0.06" radius="0.04" />
-            </geometry>
-            <material name="blue" />
-        </visual>
-        <collision>
-            <origin xyz="0.0 0 0" rpy="0 0 0"/>
-            <geometry>
-                <box size="0.12 0.15 0.15" />
-            </geometry>
-        </collision>
         <!-- <xacro:inertial_box mass="0.1" x="0.12" y="0.15" z="0.15">
             <origin xyz="0.0 0 0" rpy="0 0 0"/>
@@ -70,15 +50,4 @@
     </joint>
     <link name="lidar_link">
-        <visual>
-            <geometry>
-                <cylinder radius="0.05" length="0.04"/>
-            </geometry>
-            <material name="red"/>
-        </visual>
-        <collision>
-            <geometry>
-                <cylinder radius="0.05" length="0.04"/>
-            </geometry>
-        </collision>
         <!-- <xacro:inertial_cylinder mass="0.1" length="0.04" radius="0.05">
             <origin xyz="0 0 0" rpy="0 0 0"/>
@@ -124,4 +93,15 @@
       <child link="gps_link"/>
     </joint>
+    <!-- hydrodynamics and control plugins -->
+  <gazebo>
+    <plugin
+      filename="gz-sim-hydrodynamics-system"
+      name="gz::sim::systems::Hydrodynamics">
+      <link_name> base_link </link_name>
+      <!-- Linear and quadratic drag in heave -->
+      <zW>-5.0</zW>       <!-- Linear drag (N·s/m) -->
+      <zWabsW>-10.0</zWabsW> <!-- Quadratic drag (N·s²/m²) -->
+    </plugin>
+  </gazebo>
     </xacro:macro>
 </robot>

Commit message: Add lidar and camera sim bridge

File: stinger_description/models/stinger_base/stinger_base.xacro (robot description, xacro)
@@ -1,4 +1,5 @@
 <?xml version="1.0"?>
 <robot xmlns:xacro="http://www.ros.org/wiki/xacro" name="stinger_base">
+    <xacro:include filename="$(find stinger_description)/models/stinger_base/components/sensors.xacro"/>
     <material name="white">
       <color rgba="1 1 1 1"/>
@@ -24,4 +25,5 @@
       </collision>
       <visual name="hull_visual">
+        <origin rpy="0 0 3.1416"/>
         <geometry>
           <mesh filename="file://$(find stinger_description)/models/stinger_base/meshes/stinger_hull.dae"/>
@@ -39,24 +41,10 @@
       </visual> -->
     </link>
-    <link name="camera_link">
-        <!-- <xacro:inertial_box mass="0.1" x="0.12" y="0.15" z="0.15">
-            <origin xyz="0.0 0 0" rpy="0 0 0"/>
-        </xacro:inertial_box> -->
-    </link>
-    <joint name="camera_joint" type="fixed">
-        <origin xyz="0 0 0.1" rpy="0 0 0"/>
-        <parent link="hull_link"/>
-        <child link="camera_link"/>
-    </joint>
-    <link name="lidar_link">
-        <!-- <xacro:inertial_cylinder mass="0.1" length="0.04" radius="0.05">
-            <origin xyz="0 0 0" rpy="0 0 0"/>
-        </xacro:inertial_cylinder> -->
-    </link>
-    <joint name="lidar_joint" type="fixed">
-        <origin xyz="0 0 0.1" rpy="0 0 0"/>
-        <parent link="hull_link"/>
-        <child link="lidar_link"/>
-    </joint>
+    <xacro:camera_macro camera_id="0">
+      <origin xyz="0.1 0 0" rpy="0 0 0" />
+    </xacro:camera_macro>
+    <xacro:lidar_macro>
+      <origin xyz="0.1 0 0.1" rpy="0 0 0" />
+    </xacro:lidar_macro>
     <link name="imu_link">
       <inertial>

Commit message: Add propellers

File: stinger_description/models/stinger_base/stinger_base.xacro (robot description, xacro)
@@ -2,24 +2,16 @@
 <robot xmlns:xacro="http://www.ros.org/wiki/xacro" name="stinger_base">
     <xacro:include filename="$(find stinger_description)/models/stinger_base/components/sensors.xacro"/>
-    <material name="white">
-      <color rgba="1 1 1 1"/>
-    </material>
-    <material name="blue">
-      <color rgba="0 0 1 1"/>
-    </material>
-    <material name="red">
-      <color rgba="1 0 0 1"/>
-    </material>
+    <xacro:include filename="$(find stinger_description)/models/stinger_base/components/thrusters.xacro"/>
     <xacro:macro name="stinger_base">
     <link name="hull_link">
       <inertial>
-        <pose>-0.05 0 -0.15 0 0 0</pose>
-        <mass value="7"/>
+        <pose>0.0 0.0 -0.2 0 0 0</pose>
+        <mass value="8"/>
         <inertia ixx="2.42369" ixy="0" ixz="0" iyy="3.9235025" iyz="0" izz="5.6403125"/>
       </inertial>
       <collision>
-          <origin xyz="0 0 -0.1" rpy="0 0 0"/>
+          <origin xyz="0.0 0 -0.1" rpy="0 0 0"/>
           <geometry>
-                <box size="0.381 0.204 0.135" />
+              <box size="0.381 0.204 0.135" />
           </geometry>
       </collision>
@@ -30,24 +22,38 @@
         </geometry>
       </visual>
-      <!-- <visual name="motor_stbd_visual">
-        <geometry>
-          <mesh filename="file://$(find stinger_description)/models/stinger_base/meshes/stinger_prop.dae"/>
-        </geometry>
-      </visual>
-      <visual name="motor_port_visual">
-        <geometry>
-          <mesh filename="file://$(find stinger_description)/models/stinger_base/meshes/stinger_prop.dae"/>
-        </geometry>
-      </visual> -->
     </link>
+    <!-- Thrusters -->
+    <xacro:prop_macro thruster_id="stbd">
+      <origin xyz="-0.19 0.073 -0.041" rpy="0 0 0" />
+    </xacro:prop_macro>
+    <xacro:prop_macro thruster_id="port">
+      <origin xyz="-0.19 -0.073 -0.041 " rpy="0 0 0" />
+    </xacro:prop_macro>
+    <!-- Offset weight from propellers to maintain buoyancy -->
+    <!-- TODO: Find a better way to do this -->
+    <link name="box_offset">
+      <inertial>
+        <mass value="0.2" />
+        <origin xyz="0.19 0 0" />
+        <inertia ixx="0.2" ixy="0.0" ixz="0.0"
+                iyy="0.2" iyz="0.0"
+                izz="0.2" />
+      </inertial>
+    </link>
+    <joint name="offset_joint" type="fixed">
+      <origin xyz="0 0 0"/>
+      <parent link="hull_link"/>
+      <child link="box_offset"/>
+    </joint>
+    <!-- Sensors -->
     <xacro:camera_macro camera_id="0">
       <origin xyz="0.1 0 0" rpy="0 0 0" />
     </xacro:camera_macro>
     <xacro:lidar_macro>
-      <origin xyz="0.1 0 0.1" rpy="0 0 0" />
+      <origin xyz="0.1 0 0.025" rpy="0 0 0" />
     </xacro:lidar_macro>
     <link name="imu_link">
       <inertial>
-        <pose>0 0 0 0 0 0</pose>
+        <pose>0.1 0 0 0 0 0</pose>
         <mass value="0.1"/>
         <inertia ixx="0.0001" ixy="0" ixz="0" iyy="0.0001" iyz="0" izz="0.0001" />
@@ -65,9 +71,4 @@
     </joint>
     <link name="gps_link">
-      <inertial>
-        <pose>0 0 0 0 0 0</pose>
-        <mass value="0.1"/>
-        <inertia ixx="0.0001" ixy="0" ixz="0" iyy="0.0001" iyz="0" izz="0.0001" />
-      </inertial>
       <sensor name="gps_sensor" type="gps">
         <pose degrees="true">0 0 0 180 0 0</pose>
@@ -82,14 +83,15 @@
     </joint>
     <!-- hydrodynamics and control plugins -->
-  <gazebo>
-    <plugin
-      filename="gz-sim-hydrodynamics-system"
-      name="gz::sim::systems::Hydrodynamics">
-      <link_name> base_link </link_name>
-      <!-- Linear and quadratic drag in heave -->
-      <zW>-5.0</zW>       <!-- Linear drag (N·s/m) -->
-      <zWabsW>-10.0</zWabsW> <!-- Quadratic drag (N·s²/m²) -->
-    </plugin>
-  </gazebo>
+    <gazebo>
+      <plugin
+        filename="gz-sim-hydrodynamics-system"
+        name="gz::sim::systems::Hydrodynamics">
+        <link_name> base_link </link_name>
+        <zW>-5.0</zW>
+        <zWabsW>-10.0</zWabsW>
+        <mQ>-50.0</mQ>
+        <mQabsQ>-100.0</mQabsQ>
+      </plugin>
+    </gazebo>
     </xacro:macro>
 </robot>

Commit message: Redefine to catamaran, adjust hydrodynamic values

File: stinger_description/models/stinger_base/stinger_base.xacro (robot description, xacro)
@@ -6,6 +6,6 @@
     <link name="hull_link">
       <inertial>
-        <pose>0.0 0.0 -0.041 0 0 0</pose>
-        <mass value="8"/>
+        <pose>0.0 0.0 -0.2 0 0 0</pose>
+        <mass value="5"/>
         <inertia ixx="2.42369" ixy="0" ixz="0" iyy="3.9235025" iyz="0" izz="5.6403125"/>
       </inertial>
@@ -17,4 +17,32 @@
       </visual>
     </link>
+    <!-- port hull -->
+    <link name="hull_port_link">
+      <collision>
+          <origin xyz="0 0.0765 -0.05" rpy="0 0 0"/>
+          <geometry>
+                <box size="0.381 0.081 0.135" />
+          </geometry>
+      </collision>
+    </link>
+    <joint name="hull_port_joint" type="fixed">
+      <origin xyz="0 0 0"/>
+      <parent link="hull_link"/>
+      <child link="hull_port_link"/>
+    </joint>
+    <!-- starboard hull -->
+    <link name="hull_stbd_link">
+      <collision>
+          <origin xyz="0 -0.0765 -0.05" rpy="0 0 0"/>
+          <geometry>
+                <box size="0.381 0.081 0.135" />
+          </geometry>
+      </collision>
+    </link>
+    <joint name="hull_stbd_joint" type="fixed">
+      <origin xyz="0 0 0"/>
+      <parent link="hull_link"/>
+      <child link="hull_stbd_link"/>
+    </joint>
     <!-- Thrusters -->
     <xacro:prop_macro thruster_id="port">
@@ -100,4 +128,18 @@
         <mQ>-50.0</mQ>
         <mQabsQ>-100.0</mQabsQ>
+        <!-- Linear Drag -->
+        <xU>-5</xU> <!-- Surge -->
+        <yV>-5</yV> <!-- Sway -->
+        <zW>-5</zW> <!-- Heave -->
+        <kP>-10</kP> <!-- Roll-->
+        <mQ>-5</mQ> <!-- Pitch -->
+        <nR>-5</nR> <!-- Yaw-->
+        <xUabsU>-10</xUabsU>
+        <yVabsV>-60</yVabsV>
+        <zWabsW>-60</zWabsW>
+        <kPabsP>-10</kPabsP>
+        <mQabsQ>-60</mQabsQ>
+        <nRabsR>-50</nRabsR>
+        <default_current> 0.025 -0.025 0.5</default_current>
       </plugin>
     </gazebo>

Commit message: Remove static arg, raise lidar

File: stinger_description/models/stinger_base/stinger_base.xacro (robot description, xacro)
@@ -87,5 +87,5 @@
     </xacro:camera_macro>
     <xacro:lidar_macro>
-      <origin xyz="0.1 0 0.025" rpy="0 0 0" />
+      <origin xyz="0.1 0 0.1" rpy="0 0 0" />
     </xacro:lidar_macro>
     <xacro:imu_macro>

Commit message: Add correct IMU transform

File: stinger_description/models/stinger_base/stinger_base.xacro (robot description, xacro)
@@ -90,5 +90,5 @@
     </xacro:lidar_macro>
     <xacro:imu_macro>
-      <origin xyz="-0.05 0 0.025" rpy="0 0 0" />
+      <origin xyz="-0.05 0 0.025" rpy="3.14 0 0" />
     </xacro:imu_macro>
     <xacro:gps_macro>

Commit message: Fix typo

File: stinger_description/models/stinger_base/stinger_base.xacro (robot description, xacro)
@@ -38,5 +38,5 @@
     </joint>
     <!-- starboard hull -->
-    <link name="hull_stbd__link">
+    <link name="hull_stbd_link">
       <collision>
           <origin xyz="0.095 0 0" rpy="0 0 0"/>
@@ -52,8 +52,8 @@
       </collision>
     </link>
-    <joint name="hull_stbd__joint" type="fixed">
+    <joint name="hull_stbd_joint" type="fixed">
       <origin xyz="0.0 -0.0765 -0.035"/>
       <parent link="hull_link"/>
-      <child link="hull_stbd__link"/>
+      <child link="hull_stbd_link"/>
     </joint>
     <!-- Thrusters -->
