Commit message: fix: changed naming conventions for bridge

File: stinger_description/models/stinger_base/simulation/gz.xacro (robot description, xacro)
@@ -2,53 +2,46 @@
 <robot xmlns:xacro="http://www.ros.org/wiki/xacro">
   <gazebo>
-    <bridge>
-      <ros_topic_name>/${resolved_topic_prefix}/camera_0/image_raw</ros_topic_name>
-      <gz_topic_name>/${resolved_topic_prefix}/camera_0/image_raw</gz_topic_name>
-      <ros_type_name>sensor_msgs/msg/Image</ros_type_name>
-      <gz_type_name>gz.msgs.Image</gz_type_name>
-      <direction>GZ_TO_ROS</direction>
-    </bridge>
-    <bridge>
-      <ros_topic_name>/${resolved_topic_prefix}/laser/scan</ros_topic_name>
-      <gz_topic_name>/${resolved_topic_prefix}/laser/scan</gz_topic_name>
-      <ros_type_name>sensor_msgs/msg/LaserScan</ros_type_name>
-      <gz_type_name>gz.msgs.LaserScan</gz_type_name>
-      <direction>GZ_TO_ROS</direction>
-    </bridge>
-    <bridge>
-      <ros_topic_name>/${resolved_topic_prefix}/imu/data</ros_topic_name>
-      <gz_topic_name>/${resolved_topic_prefix}/imu/data</gz_topic_name>
-      <ros_type_name>sensor_msgs/msg/Imu</ros_type_name>
-      <gz_type_name>gz.msgs.IMU</gz_type_name>
-      <direction>GZ_TO_ROS</direction>
-    </bridge>
-    <bridge>
-      <ros_topic_name>/${resolved_topic_prefix}/gps/fix</ros_topic_name>
-      <gz_topic_name>/${resolved_topic_prefix}/gps/fix</gz_topic_name>
-      <ros_type_name>sensor_msgs/msg/NavSatFix</ros_type_name>
-      <gz_type_name>gz.msgs.NavSat</gz_type_name>
-      <direction>GZ_TO_ROS</direction>
-    </bridge>
-    <bridge>
-      <ros_topic_name>/${resolved_topic_prefix}/thruster_port/cmd_thrust</ros_topic_name>
-      <gz_topic_name>/model/${model_name}/joint/${frame_prefix}prop_joint_port/cmd_thrust</gz_topic_name>
-      <ros_type_name>std_msgs/msg/Float64</ros_type_name>
-      <gz_type_name>gz.msgs.Double</gz_type_name>
-      <direction>ROS_TO_GZ</direction>
-    </bridge>
-    <bridge>
-      <ros_topic_name>/${resolved_topic_prefix}/thruster_stbd/cmd_thrust</ros_topic_name>
-      <gz_topic_name>/model/${model_name}/joint/${frame_prefix}prop_joint_stbd/cmd_thrust</gz_topic_name>
-      <ros_type_name>std_msgs/msg/Float64</ros_type_name>
-      <gz_type_name>gz.msgs.Double</gz_type_name>
-      <direction>ROS_TO_GZ</direction>
-    </bridge>
-    <bridge>
-      <ros_topic_name>/ground_truth/${model_name}/odometry</ros_topic_name>
-      <gz_topic_name>/model/${model_name}/odometry_with_covariance</gz_topic_name>
-      <ros_type_name>nav_msgs/msg/Odometry</ros_type_name>
-      <gz_type_name>gz.msgs.OdometryWithCovariance</gz_type_name>
-      <direction>GZ_TO_ROS</direction>
-    </bridge>
+    <bridge
+      ros_topic="/${resolved_topic_prefix}/camera_0/image_raw"
+      gz_topic="/${resolved_topic_prefix}/camera_0/image_raw"
+      ros_type="sensor_msgs/msg/Image"
+      gz_type="gz.msgs.Image"
+      direction="gz_to_ros"/>
+    <bridge
+      ros_topic="/${resolved_topic_prefix}/laser/scan"
+      gz_topic="/${resolved_topic_prefix}/laser/scan"
+      ros_type="sensor_msgs/msg/LaserScan"
+      gz_type="gz.msgs.LaserScan"
+      direction="gz_to_ros"/>
+    <bridge
+      ros_topic="/${resolved_topic_prefix}/imu/data"
+      gz_topic="/${resolved_topic_prefix}/imu/data"
+      ros_type="sensor_msgs/msg/Imu"
+      gz_type="gz.msgs.IMU"
+      direction="gz_to_ros"/>
+    <bridge
+      ros_topic="/${resolved_topic_prefix}/gps/fix"
+      gz_topic="/${resolved_topic_prefix}/gps/fix"
+      ros_type="sensor_msgs/msg/NavSatFix"
+      gz_type="gz.msgs.NavSat"
+      direction="gz_to_ros"/>
+    <bridge
+      ros_topic="/${resolved_topic_prefix}/thruster_port/cmd_thrust"
+      gz_topic="/model/${model_name}/joint/${frame_prefix}prop_joint_port/cmd_thrust"
+      ros_type="std_msgs/msg/Float64"
+      gz_type="gz.msgs.Double"
+      direction="ros_to_gz"/>
+    <bridge
+      ros_topic="/${resolved_topic_prefix}/thruster_stbd/cmd_thrust"
+      gz_topic="/model/${model_name}/joint/${frame_prefix}prop_joint_stbd/cmd_thrust"
+      ros_type="std_msgs/msg/Float64"
+      gz_type="gz.msgs.Double"
+      direction="ros_to_gz"/>
+    <bridge
+      ros_topic="/ground_truth/${model_name}/odometry"
+      gz_topic="/model/${model_name}/odometry_with_covariance"
+      ros_type="nav_msgs/msg/Odometry"
+      gz_type="gz.msgs.OdometryWithCovariance"
+      direction="gz_to_ros"/>
   </gazebo>
 </robot>

File: stinger_description/urdf/stinger_tug.urdf.xacro (robot description, xacro)
@@ -4,7 +4,7 @@
   <xacro:arg name="namespace" default="__default__"/>
   <xacro:arg name="topic_prefix" default="__default__"/>
-  <xacro:property name="frame_prefix" value="$(eval arg('prefix') if arg('prefix') != '__default__' else (arg('namespace') + '_' if arg('namespace') != '__default__' else ''))"/>
-  <xacro:property name="resolved_topic_prefix" value="$(eval arg('topic_prefix') if arg('topic_prefix') != '__default__' else (arg('namespace') if arg('namespace') != '__default__' else 'stinger'))"/>
-  <xacro:property name="model_name" value="$(eval arg('namespace') + '_stinger_tug' if arg('namespace') != '__default__' else 'stinger')"/>
+  <xacro:property name="frame_prefix" value="${xacro.arg('prefix') if xacro.arg('prefix') != '__default__' else xacro.arg('namespace') + '_' if xacro.arg('namespace') != '__default__' else ''}"/>
+  <xacro:property name="resolved_topic_prefix" value="${xacro.arg('topic_prefix') if xacro.arg('topic_prefix') != '__default__' else xacro.arg('namespace') if xacro.arg('namespace') != '__default__' else 'stinger'}"/>
+  <xacro:property name="model_name" value="${xacro.arg('namespace') + '_stinger_tug' if xacro.arg('namespace') != '__default__' else 'stinger'}"/>
   <xacro:include filename="$(find stinger_description)/models/stinger_base/simulation/gz.xacro"/>
   <xacro:include filename="$(find stinger_description)/models/stinger_base/stinger_base.xacro"/>
